Commit message: Updates to files after reorganization
Updated urdf file for built vehicle

File: houseRobo_ros1_ws/src/houseRobo_package/urdf/simple_houseRobo.urdf (robot description, URDF)
Before this commit: robot house_robot, 2 links, 1 joints
Joints:
- joint laser_joint: origin xyz=0 0 0.04 rpy=0 0 0 -> xyz=0.065 0 0.13 rpy=0 0 0

Commit message: Changed laser_link to laser as it is required for slam_gmapping

File: houseRobo_ros1_ws/src/houseRobo_package/urdf/simple_houseRobo.urdf (robot description, URDF)
Before this commit: robot house_robot, 2 links, 1 joints
Links:
- removed link laser_link
- added link laser
Joints:
- joint laser_joint: child laser_link -> laser
